File: Hardware/GPIO_Block.sch (EAGLE design)
At the start: 20 parts, among them U1 TXB0108, U2 EDISON_CONNECTOR_FULLMOUNTING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, U3 EDISON_CONNECTOR_FULLHEADER, U4 TXB0108

Commit message: t/bRestrict between connector pads. (v10)
Other:
- note added: "v10"
- note removed: "v02"
Changed lines of the file:
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@@
 <?xml version="1.0" encoding="utf-8"?>
 <!DOCTYPE eagle SYSTEM "eagle.dtd">
-<eagle version="6.5.0">
+<eagle version="7.1.0">
 <drawing>
 <settings>
@@
 <sheet>
 <plain>
-<text x="238.76" y="7.62" size="2.54" layer="94">v02</text>
+<text x="238.76" y="7.62" size="2.54" layer="94">v10</text>
 <text x="167.64" y="7.62" size="2.54" layer="94">Casey Kuhns</text>
 </plain>
